File: rp2040.kicad_sch (KiCad schematic)
At the start: 43 parts, among them U1 GT-USB-7010AN

Commit message: small rp2040 changes and the cypd3177
Parts:
- removed SW?: Latching, easyeda2kicad:SW-TH_6P-L8.0-W8.0-P2.50, symbol Switch:SW_Push
Changed lines of the file:
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@@
 	)
 	(junction
-		(at 252.73 116.84)
-		(diameter 0)
-		(color 0 0 0 0)
-	)
-	(junction
 		(at 38.1 115.57)
 		(diameter 0)
@@
 	(wire
 		(pts
-			(xy 227.33 111.76) (xy 234.95 111.76)
-		)
-		(stroke
-			(width 0)
-			(type default)
-		)
-	)
-	(wire
-		(pts
 			(xy 217.17 26.67) (xy 227.33 26.67)
 		)
@@
 	(wire
 		(pts
-			(xy 245.11 111.76) (xy 252.73 111.76)
-		)
-		(stroke
-			(width 0)
-			(type default)
-		)
-	)
-	(wire
-		(pts
 			(xy 247.65 129.54) (xy 252.73 129.54)
 		)
@@
 	(wire
 		(pts
-			(xy 252.73 111.76) (xy 252.73 116.84)
-		)
-		(stroke
-			(width 0)
-			(type default)
-		)
-	)
-	(wire
-		(pts
 			(xy 227.33 114.3) (xy 261.62 114.3)
 		)
@@
 					(unit 1)
 				)
-			)
-		)
-	)
-	(symbol
-		(lib_id "Switch:SW_Push")
-		(at 240.03 111.76 0)
-		(unit 1)
-		(exclude_from_sim no)
-		(in_bom yes)
-		(on_board yes)
-		(dnp no)
-		(property "Reference" "SW?"
-			(at 235.712 110.49 0)
-			(effects
-				(font
-					(size 1.016 1.016)
-				)
-			)
-		)
-		(property "Value" "Latching"
-			(at 245.872 110.49 0)
-			(effects
-				(font
-					(size 1.016 1.016)
-				)
-			)
-		)
-		(property "Footprint" "easyeda2kicad:SW-TH_6P-L8.0-W8.0-P2.50"
-			(at 240.03 106.68 0)
-			(effects
-				(font
-					(size 1.27 1.27)
-				)
-				(hide yes)
-			)
-		)
-		(property "Datasheet" "~"
-			(at 240.03 106.68 0)
-			(effects
-				(font
-					(size 1.27 1.27)
-				)
-				(hide yes)
-			)
-		)
-		(property "Description" "Push button switch, generic, two pins"
-			(at 240.03 111.76 0)
-			(effects
-				(font
-					(size 1.27 1.27)
-				)
-				(hide yes)
-			)
-		)
-		(pin "1"
-		)
-		(pin "2"
-		)
-		(instances
-			(project "raspberry-pi-power-hub"
-				(path "/2a0acc6a-7dcb-4f06-b9d0-ff1420b61fe9/c01414cb-6643-43a4-b4a5-f11e07d2900d"
-					(reference "SW?")
-					(unit 1)
-				)

Commit message: peak schematic
Parts:
- removed D?: 200V,20A, Diode_SMD:D_SMB_Handsoldering, symbol Device:D_Schottky
- added C1: 220uF, symbol Device:C_Polarized_Small
- added C2: 1000uF, symbol Device:C_Polarized_Small
- added D1, D2, D3: 200V,20A, symbol Device:D_Schottky_Small
- added L1: 47uH, easyeda2kicad:IND-SMD_L7.2-W6.6_GPSR07X0, symbol Device:L_Small
- added U4: SXL1509-3.3E1, easyeda2kicad:SOP-8_L4.9-W3.9-P1.27-LS6.0-BL-1, symbol easyeda2kicad:SXL1509-3.3E1
Connections:
- net +3.3V: now also C1.1, L1.2, U4.3 (FB)
- net GND: now also C1.2, C2.2, D3.2 (A), U4.5 (GND), U4.6 (GND), U4.7 (GND), U4.8 (GND)
- net VBUS: now also D1.2 (A), D2.2 (A)
- net +1V1 renamed +1.1V
- new net: C2.1, D1.1 (K), D2.1 (K), U4.1 (VIN), U4.4 (EN)
- new net: D3.1 (K), L1.1, U4.2 (OUTPUT)
Other:
- note added: "same diode"

Commit message: owo
Parts:
- removed C1: 220uF, symbol Device:C_Polarized_Small
- removed C2: 1000uF, symbol Device:C_Polarized_Small
- removed D1, D2, D3: 200V,20A, symbol Device:D_Schottky_Small
- removed U4: SXL1509-3.3E1, easyeda2kicad:SOP-8_L4.9-W3.9-P1.27-LS6.0-BL-1, symbol easyeda2kicad:SXL1509-3.3E1
- removed U?: ABM8-272-T3_C20625731, easyeda2kicad:CRYSTAL-SMD_4P-L3.2-W2.5-BL, symbol EasyEDA:ABM8-272-T3_C20625731
- added C1, C2: 22uF, symbol Device:C_Small
- added C11: 0.1uF, Capacitor_SMD:C_0402_1005Metric, symbol Device:C_Small
- added C3: 10uF, symbol Device:C_Small
- added D4, D5: 200V,20A, symbol Device:D_Schottky_Small
- added JP1: SolderJumper_2_Bridged, Jumper:SolderJumper-2_P1.3mm_Bridged_RoundedPad1.0x1.5mm, symbol Jumper:SolderJumper_2_Bridged
- added U6: AP63203WU-7, AP63203WU-7_DIO, symbol AP63203WU_7:AP63203WU-7
- added U7: ABM8-272-T3_C20625731, easyeda2kicad:CRYSTAL-SMD_4P-L3.2-W2.5-BL, symbol easyeda2kicad:ABM8-272-T3_C20625731
- L1: value 47uH -> 4.7uH; footprint easyeda2kicad:IND-SMD_L7.2-W6.6_GPSR07X0 -> easyeda2kicad:IND-SMD_L5.4-W5.2_CMLE051E
Connections:
- net +3.3V: now also C1.1, C2.1, U6.1 (FB)
- net GND: now also C1.2, C2.2, C3.2, U6.4 (GND), U7.2 (GND), U7.4 (GND)
- net VBUS: now also D4.2 (A); no longer U1.A4B9 (VBUS), U1.B4A9 (VBUS)
- net XIN: now also U7.1
- net at C?.2, R?.1: now also U7.3
- net at L1.1: now also C11.2, U6.5 (SW)
- new net: JP1.2 (B), U6.2 (EN)
- new net: C3.1, D4.1 (K), D5.1 (K), JP1.1 (A), U6.3 (VIN)
- new net: C11.1, U6.6 (BST)
- new net USB_VBUS: D5.2 (A), U1.A4B9 (VBUS), U1.B4A9 (VBUS)
Other:
- moved on the sheet: C?, L1

Commit message: finished pcb routing yay
Parts:
- removed D4, D5: 200V,20A, symbol Device:D_Schottky_Small
- removed R?: 10k, Resistor_SMD:R_0402_1005Metric_Pad0.72x0.64mm_HandSolder, symbol Device:R_Small
- removed R? (x2): 5.1k, Resistor_SMD:R_0402_1005Metric_Pad0.72x0.64mm_HandSolder, symbol Device:R_Small
- removed R?: 470, Resistor_SMD:R_0402_1005Metric_Pad0.72x0.64mm_HandSolder, symbol Device:R_Small
- removed U1: GT-USB-7010AN, easyeda2kicad:USB-SMD_GT-USB-7010AN, symbol easyeda2kicad:GT-USB-7010AN
- added TP1, TP10, TP11, TP12, TP13, TP14, TP15, TP16, TP17, TP18, TP19, TP2, TP20, TP21, TP22, TP23, TP3, TP4, TP5, TP6, TP7, TP8, TP9: TestPoint, TestPoint:TestPoint_Pad_D1.5mm, symbol Connector:TestPoint
- C1, C11, C12, C13, C2, C4, C5, C6, C7, C8, C9: renamed from C?; footprint Capacitor_SMD:C_0201_0603Metric_Pad0.64x0.40mm_HandSolder -> Capacitor_SMD:C_0402_1005Metric
- C10, C3: renamed from C?; footprint Capacitor_SMD:C_0402_1005Metric_Pad0.74x0.62mm_HandSolder -> Capacitor_SMD:C_0603_1608Metric
- C14: renamed from C11; value 0.1uF -> 100nF
- C15: renamed from C3; footprint (none) -> Capacitor_SMD:C_0805_2012Metric
- C16: renamed from C1; footprint (none) -> Capacitor_SMD:C_0603_1608Metric
- C17: renamed from C2; footprint (none) -> Capacitor_SMD:C_0603_1608Metric
- U5: renamed from U6; footprint AP63203WU-7_DIO -> AP63203WU_7:AP63203WU-7_DIO
- gave numbers to parts that had none: 22
- renumbered U7 to U3
Connections:
- net USB_R_D+ is gone; now on net USB_D+: R3.1
- net USB_R_D- is gone; now on net USB_D-: R4.1
- net GPIO0: now also TP1.1
- net GPIO1: now also TP2.1
- net GPIO10: now also TP11.1
- net GPIO11: now also TP12.1
- net GPIO12: now also TP13.1
- net GPIO13: now also TP14.1
- net GPIO14: now also TP15.1
- net GPIO2: now also TP3.1
- net GPIO26: now also TP20.1
- net GPIO27: now also TP21.1
- net GPIO28: now also TP22.1
- net GPIO29: now also TP23.1
- net GPIO3: now also TP4.1
- net GPIO4: now also TP5.1
- net GPIO5: now also TP6.1
- net GPIO6: now also TP7.1
- net GPIO7: now also TP8.1
- net GPIO8: now also TP9.1
- net GPIO9: now also TP10.1
- net SCL: now also TP18.1
- net SDA: now also TP17.1
- net USB_D+: no longer R3.2, U4.47 (USB_DP)
- net USB_D-: no longer R4.2, U4.46 (USB_DM)
- net VBUS: now also C15.1, JP1.1 (A), U5.3 (VIN)
- net GPIO15: now reaches U4.18 (GPIO15)
- net GPIO15: now also TP16.1
- net GPIO18: now reaches U4.29 (GPIO18)
- net GPIO18: now also TP19.1
- new net LUSB_D+: R3.2, U4.47 (USB_DP)
- new net LUSB_D-: R4.2, U4.46 (USB_DM)
Other:
- note removed: "same diode"
