File: usb_pwr_in.kicad_sch (KiCad schematic)
At the start: 1 part, among them U2 CYPD3177-24LQ

Commit message: peak schematic
Parts:
- added U3: GT-USB-7010AN, easyeda2kicad:USB-SMD_GT-USB-7010AN, symbol easyeda2kicad:GT-USB-7010AN
Connections:
- net GND: now reaches U2.19 (GND), U2.22 (GND), U2.25 (GND)
- new net: U3.13 (GND), U3.14 (GND), U3.15 (GND), U3.16 (GND), U3.A1B12 (GND), U3.B1A12 (GND)
- new net: U3.A4B9 (VBUS), U3.B4A9 (VBUS)
Changed lines of the file:
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@@
+		)
+	)
+	(symbol
+		(lib_id "easyeda2kicad:GT-USB-7010AN")
+		(at 39.37 109.22 0)
+		(unit 1)
+		(exclude_from_sim no)
+		(in_bom yes)
+		(on_board yes)
+		(dnp no)
+		(fields_autoplaced yes)
+		(property "Reference" "U3"
+			(at 39.37 91.44 0)
+			(effects
+				(font
+					(size 1.27 1.27)
+				)
+			)
+		)
+		(property "Value" "GT-USB-7010AN"
+			(at 39.37 95.25 0)
+			(effects
+				(font
+					(size 1.27 1.27)
+				)
+			)
+		)
+		(property "Footprint" "easyeda2kicad:USB-SMD_GT-USB-7010AN"
+			(at 39.37 128.27 0)
+			(effects
+				(font
+					(size 1.27 1.27)
+				)
+				(hide yes)
+			)
+		)
+		(property "Datasheet" ""
+			(at 39.37 109.22 0)
+			(effects
+				(font
+					(size 1.27 1.27)
+				)
+				(hide yes)
+			)
+		)
+		(property "Description" ""
+			(at 39.37 109.22 0)
+			(effects
+				(font
+					(size 1.27 1.27)
+				)
+				(hide yes)
+			)
+		)
+		(property "LCSC Part" "C963370"
+			(at 39.37 128.27 0)
+			(effects
+				(font
+					(size 1.27 1.27)
+				)
+				(hide yes)
+			)
+		)
+		(pin "A4B9"
+		)
+		(pin "A7"
+		)
+		(pin "A5"
+		)
+		(pin "B7"
+		)
+		(pin "B4A9"
+		)
+		(pin "16"
+		)
+		(pin "A1B12"
+		)
+		(pin "14"
+		)
+		(pin "B5"
+		)
+		(pin "A6"
+		)
+		(pin "15"
+		)
+		(pin "B8"
+		)
+		(pin "A8"
+		)
+		(pin "13"
+		)
+		(pin "B1A12"
+		)
+		(pin "B6"
+		)
+		(instances
+			(project ""
+				(path "/2a0acc6a-7dcb-4f06-b9d0-ff1420b61fe9/2f555ee9-9c04-4335-99e6-65577b3bf6f3"
+					(reference "U3")
+					(unit 1)
+				)
+			)
+		)
+	)
+	(symbol
+		(lib_id "power:GND")
+		(at 109.22 130.81 0)
+		(unit 1)
+		(exclude_from_sim no)
+		(in_bom yes)
+		(on_board yes)
+		(dnp no)
+		(fields_autoplaced yes)
+		(property "Reference" "#PWR01"
+			(at 109.22 137.16 0)
+			(effects
+				(font
+					(size 1.27 1.27)
+				)
+				(hide yes)
+			)
+		)
+		(property "Value" "GND"
+			(at 109.22 135.89 0)
+			(effects
+				(font
+					(size 1.27 1.27)
+				)
+			)
+		)
+		(property "Footprint" ""
+			(at 109.22 130.81 0)
+			(effects
+				(font
+					(size 1.27 1.27)
+				)
+				(hide yes)
+			)
+		)
+		(property "Datasheet" ""
+			(at 109.22 130.81 0)
+			(effects
+				(font
+					(size 1.27 1.27)
+				)
+				(hide yes)
+			)
+		)
+		(property "Description" "Power symbol creates a global label with name \"GND\" , ground"
+			(at 109.22 130.81 0)
+			(effects
+				(font
+					(size 1.27 1.27)
+				)
+				(hide yes)
+			)
+		)
+		(pin "1"
+		)
+		(instances
+			(project ""
+				(path "/2a0acc6a-7dcb-4f06-b9d0-ff1420b61fe9/2f555ee9-9c04-4335-99e6-65577b3bf6f3"
+					(reference "#PWR01")
+					(unit 1)
+				)
+			)
 		)
 	)

Commit message: owo
Parts:
- added C10, C9: 1uF, symbol Device:C
- added C4, C8: 1uF, Capacitor_SMD:C_0402_1005Metric_Pad0.74x0.62mm_HandSolder, symbol Device:C_Small
- added C5: 4.7uF, symbol Device:C
- added C6, C7: 100nF, Capacitor_SMD:C_0201_0603Metric_Pad0.64x0.40mm_HandSolder, symbol Device:C_Small
- added D1, D2: D_Zener, Diode_SMD:D_SOD-123, symbol Device:D_Zener
- added D3: Red, symbol Device:LED
- added Q1, Q2: AOD409-HXY, easyeda2kicad:TO-252-2_L6.6-W6.1-P4.57-LS9.9-TL-CW, symbol easyeda2kicad:AOD409-HXY
- added Q3: NPN, symbol Simulation_SPICE:NPN
- added R1: 4.7k, symbol Device:R
- added R2, R6: 1k, symbol Device:R
- added R3: 49.9k, symbol Device:R
- added R4: 10k, symbol Device:R
- added R5: 470, symbol Device:R
- added R7: 5.1k, symbol Device:R
Connections:
- net GND: now also U2.1 (VBUS_MIN), U2.6 (ISNK_FINE), U3.13 (GND), U3.14 (GND), U3.15 (GND), U3.16 (GND), U3.A1B12 (GND), U3.B1A12 (GND), C4.2, C5.2, C6.1, C7.1, C8.1, D3.1 (K), R6.1
- net at U2.10 (FLIP): now also R1.1
- net VBUS: now reaches U2.11 (VDC_OUT)
- net VBUS: now also C10.1, Q2.2 (D)
- net SCL: now reaches U2.12 (HPI_SDA)
- net SDA: now reaches U2.13 (HPI_SCL)
- net at U2.14 (CC2): now also U3.B5 (CC2)
- net at U2.15 (CC1): now also U3.A5 (CC1)
- net USB_VBUS: now reaches U2.18 (VBUS_IN)
- net USB_VBUS: now also U3.A4B9 (VBUS), U3.B4A9 (VBUS), C5.1, C9.1, Q1.2 (D), Q3.1 (C), R4.2
- net 3.3V+: now reaches U2.2 (VBUS_MAX)
- net 3.3V+: now also U2.23 (VDDD), C6.2, C7.2, C8.2, R1.2, R7.2
- net at U2.24 (VCCD): now also C4.1
- net at U2.3 (VBUS_FET_EN): now also R2.1
- net at U2.5 (ISNK_COARSE): now also R6.2, R7.1
- net at U2.9 (FAULT): now also Q3.2 (B)
- new net: C10.2, C9.2, D1.2 (A), D2.2 (A), R2.2, R3.1, R4.1
- new net: D2.1 (K), Q2.1 (G)
- new net: D3.2 (A), R5.1
- new net: D1.1 (K), Q1.1 (G)
- new net: Q1.3 (S), Q2.3 (S), R3.2
- new net: Q3.3 (E), R5.2
- no-connect marks 0 -> 3
Other:
- moved on the sheet: U3

Commit message: finished pcb routing yay
Parts:
- C18: renamed from C6; footprint Capacitor_SMD:C_0201_0603Metric_Pad0.64x0.40mm_HandSolder -> Capacitor_SMD:C_0402_1005Metric
- C19: renamed from C7; footprint Capacitor_SMD:C_0201_0603Metric_Pad0.64x0.40mm_HandSolder -> Capacitor_SMD:C_0402_1005Metric
- C20: renamed from C8; footprint Capacitor_SMD:C_0402_1005Metric_Pad0.74x0.62mm_HandSolder -> Capacitor_SMD:C_0603_1608Metric
- C21: renamed from C4; footprint Capacitor_SMD:C_0402_1005Metric_Pad0.74x0.62mm_HandSolder -> Capacitor_SMD:C_0603_1608Metric
- C22: renamed from C5; footprint (none) -> Capacitor_SMD:C_1206_3216Metric
- C23: renamed from C9; footprint (none) -> Capacitor_SMD:C_0603_1608Metric
- C24: renamed from C10; footprint (none) -> Capacitor_SMD:C_0603_1608Metric
- D11: renamed from D3; footprint (none) -> LED_SMD:LED_0603_1608Metric_Pad1.05x0.95mm_HandSolder
- Q3: footprint (none) -> Package_TO_SOT_SMD:SOT-23
- R16: renamed from R1; footprint (none) -> Resistor_SMD:R_0402_1005Metric_Pad0.72x0.64mm_HandSolder
- R17: renamed from R4; footprint (none) -> Resistor_SMD:R_0402_1005Metric_Pad0.72x0.64mm_HandSolder
- R18: renamed from R3; footprint (none) -> Resistor_SMD:R_0402_1005Metric_Pad0.72x0.64mm_HandSolder
- R19: renamed from R7; footprint (none) -> Resistor_SMD:R_0402_1005Metric_Pad0.72x0.64mm_HandSolder
- R20: renamed from R2; footprint (none) -> Resistor_SMD:R_0402_1005Metric_Pad0.72x0.64mm_HandSolder
- R21: renamed from R6; footprint (none) -> Resistor_SMD:R_0402_1005Metric_Pad0.72x0.64mm_HandSolder
- R22: renamed from R5; footprint (none) -> Resistor_SMD:R_0402_1005Metric_Pad0.72x0.64mm_HandSolder
- renumbered D2 to D10, D1 to D9, U2 to U6, U3 to U7
Connections:
- net USB_D+: now reaches U7.A6 (DP1)
- net USB_D+: now also U7.B6 (DP2)
- net USB_D-: now reaches U7.A7 (DN1)
- net USB_D-: now also U7.B7 (DN2)
